File: ArenaTimer/ArenaTimer.kicad_pcb (KiCad board)
At the start: 2 copper layers, 262.2 x 230 mm, 200 parts, among them J1 Blue ready-up, J10 Red ready-up, J11 Bell Power, J12 Screw_Terminal_01x03, J13 Screw_Terminal_01x03, J15 Conn_01x15_Socket, J16 Conn_01x15_Socket, J2 Conn_01x02_Socket, J3 Conn_01x02_Pin, J4 GND, J5 5V, J6 GND, J7 5V, J8 Barrel_Jack, J9 Conn_01x06_Pin, K1 G5V-2_Split, Q1 BSS214NW

Commit message: update board for next order
Parts:
- removed J11: Bell Power, TerminalBlock:TerminalBlock_bornier-2_P5.08mm
- removed JP1: Jumper_2_Open, Jumper:SolderJumper-2_P1.3mm_Open_RoundedPad1.0x1.5mm
- added C1: 100nF, Capacitor_SMD:C_0402_1005Metric, F.Cu at (255.8, 251.2)
- added C2: 100nF, Capacitor_SMD:C_0402_1005Metric, F.Cu at (258.3, 251.2)
- added C3: 100nF, Capacitor_SMD:C_0402_1005Metric, F.Cu at (260.8, 251.2)
- added C4: 100nF, Capacitor_SMD:C_0402_1005Metric, F.Cu at (263.3, 251.2)
- added C5: 100nF, Capacitor_SMD:C_0402_1005Metric, F.Cu at (265.8, 251.2)
- added C6: 100nF, Capacitor_SMD:C_0402_1005Metric, F.Cu at (239.4, 251.3)
- added C7: 100nF, Capacitor_SMD:C_0402_1005Metric, F.Cu at (221.2, 251.2)
- added J14: WAGO, WAGO_2060-452_998-404:2060-452_998-404, B.Cu at (249.7, 77.5)
- added R3: 10k, Resistor_SMD:R_0402_1005Metric, F.Cu at (256.9, 251.2)
- added R4: 10k, Resistor_SMD:R_0402_1005Metric, F.Cu at (259.4, 251.2)
- added R5: 10k, Resistor_SMD:R_0402_1005Metric, F.Cu at (261.9, 251.2)
- added R6: 10k, Resistor_SMD:R_0402_1005Metric, F.Cu at (264.4, 251.2)
- added R7: 10k, Resistor_SMD:R_0402_1005Metric, F.Cu at (266.9, 251.2)
- added R8: 10k, Resistor_SMD:R_0402_1005Metric, F.Cu at (238.3, 251.3)
- added R9: 10k, Resistor_SMD:R_0402_1005Metric, F.Cu at (220.1, 251.2)
- J13: value Screw_Terminal_01x03 -> WAGO; footprint TerminalBlock:TerminalBlock_bornier-3_P5.08mm -> WAGO_2060-452_998-404:2060-452_998-404
- J8: value Barrel_Jack -> PJ-082BH; footprint Connector_BarrelJack:BarrelJack_Horizontal -> SAMESKY_PJ-082BH:SAMESKY_PJ-082BH; moved to F.Cu
- moved J13 184.4 mm to (237.8, 54.0)
- moved J12 18.6 mm to (56.1, 29.2)
- moved J8 9.25 mm to (61.5, 252.7), turned to 0 degrees
- moved D8 0.98 mm to (71.1, 247.1)
- moved J16 0.05 mm to (122.8, 190.3)
Connections:
- J12 pad 3: GND -> Net-(J12-Pin_3)
- J13 pad 1: Net-(J13-Pin_1) -> +5V
- J13 pad 2: Net-(J13-Pin_2) -> GND
- J15 pad 10: nSTART_BTN -> nRED_RDY_BTN
- J15 pad 11: nPAUSE_BTN -> nBLUE_RDY_BTN
- J15 pad 12: nRESET_BTN -> nBUZZER_BTN
- J15 pad 13: nTIME_SEL -> unconnected-(J15-Pin_13-Pad13)
- J15 pad 15: +5V -> +3.3V
- J15 pad 8: unconnected-(J15-Pin_8-Pad8) -> DIGIT_LEDS
- J15 pad 9: unconnected-(J15-Pin_9-Pad9) -> BORDER_LEDS
- J16 pad 10: nRIGHT_RDY_BTN -> nSTART_BTN
- J16 pad 11: nLEFT_RDY_BTN -> nPAUSE_BTN
- J16 pad 12: nBUZZER_BTN -> nRESET_BTN
- J16 pad 13: RELAY_EN -> nTIME_SEL
- J16 pad 15: +3.3V -> +5V
- J16 pad 8: DIGIT_LEDS -> unconnected-(J16-Pin_8-Pad8)
- J16 pad 9: BORDER_LEDS -> unconnected-(J16-Pin_9-Pad9)
- J3 pad 1: /TimerColon/DOUT -> /TimerBorder/DOUT
- J3 pad 2: /TimerBorder/DOUT -> /TimerColon/DOUT
- K1 pad 11: Net-(J13-Pin_1) -> (no net)
- K1 pad 13: Net-(J11-Pin_1) -> (no net)
- K1 pad 4: Net-(J11-Pin_1) -> Net-(J12-Pin_3)
- K1 pad 9: Net-(J13-Pin_2) -> (no net)
Routing:
- net +3.3V: track 0.00 -> 272.4 mm, vias 0 -> 3
- net nRED_RDY_BTN: track 0.00 -> 231.2 mm, vias 0 -> 2
- net nBLUE_RDY_BTN: track 0.00 -> 211.7 mm, vias 0 -> 2
- net Net-(J11-Pin_1): track 59.7 -> 0.00 mm
- net Net-(J12-Pin_3): track 0.00 -> 45.1 mm
- net Net-(J13-Pin_1): track 40.9 -> 0.00 mm
- net Net-(J13-Pin_2): track 34.3 -> 0.00 mm
- net nRESET_BTN: track 246.0 -> 220.1 mm
- net nPAUSE_BTN: track 241.2 -> 216.4 mm
- net nBUZZER_BTN: track 224.9 -> 248.4 mm
- net nSTART_BTN: track 237.5 -> 215.6 mm
- net BORDER_LEDS: track 358.3 -> 338.6 mm, vias 3 -> 2
- net nTIME_SEL: track 248.6 -> 230.0 mm
- net DIGIT_LEDS: track 331.3 -> 321.4 mm
- net Net-(J12-Pin_2): track 40.6 -> 32.9 mm
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- added copper zone on B.Cu, net +5V
Other:
- board text added: "COM"
- board text added: "SEMO Combat Robotics 2026 Vinnie Marco"
- board text removed: "SEMO Combat Robotics 2025 Vinnie Marco Mitch Cerroni"
- board text removed: "Short JP1 for 5V buzzer power"
- board text removed: "V+"
