File: ArenaTimer/ArenaTimer.kicad_sch (KiCad schematic)
At the start: 29 parts, among them J1 Blue ready-up, J10 Red ready-up, J11 Bell Power, J12 Screw_Terminal_01x03, J13 Screw_Terminal_01x03, J15 Conn_01x15_Socket, J16 Conn_01x15_Socket, J2 Conn_01x02_Socket, J3 Conn_01x02_Pin, J4 GND, J5 5V, J6 GND, J7 5V, J8 Barrel_Jack, J9 Conn_01x06_Pin, K1 G5V-2_Split, Q1 BSS214NW

Commit message: update board for next order
Parts:
- removed J11: Bell Power, TerminalBlock:TerminalBlock_bornier-2_P5.08mm, symbol Connector:Screw_Terminal_01x02
- removed J13: Screw_Terminal_01x03, TerminalBlock:TerminalBlock_bornier-3_P5.08mm, symbol Connector:Screw_Terminal_01x03
- removed J8: Barrel_Jack, Connector_BarrelJack:BarrelJack_Horizontal, symbol Connector:Barrel_Jack
- removed JP1: Jumper_2_Open, Jumper:SolderJumper-2_P1.3mm_Open_RoundedPad1.0x1.5mm, symbol Jumper:Jumper_2_Open
- removed unit 3 of K1
- added C1, C2, C3, C4, C5, C6, C7: 100nF, Capacitor_SMD:C_0402_1005Metric, symbol Device:C
- added J13, J14: WAGO, WAGO_2060-452_998-404:2060-452_998-404, symbol Connector:Conn_01x02_Socket
- added J8: PJ-082BH, SAMESKY_PJ-082BH:SAMESKY_PJ-082BH, symbol PJ-082BH:PJ-082BH
- added R3, R4, R5, R6, R7, R8, R9: 10k, Resistor_SMD:R_0402_1005Metric, symbol Device:R_US
- J1, J10, J15, J16: now fitted; now in the parts list
- J12: LCSC (none) -> C72334
- J2: LCSC (none) -> C2897384; now fitted; now in the parts list
- J3: LCSC (none) -> C492410; now fitted; now in the parts list
- J4, J5: LCSC (none) -> C492412; now fitted; now in the parts list
- J6, J7: LCSC C5142237 -> C2897386; now fitted; now in the parts list
- J9: LCSC (none) -> C157919; now fitted; now in the parts list
Connections:
- net +3.3V: now also J15.15 (Pin_15), R3.1, R4.1, R5.1, R6.1, R7.1, R8.1, R9.1; no longer J16.15 (Pin_15)
- net +5V: now also J16.15 (Pin_15), J13.1 (Pin_1), J8.1; no longer J15.15 (Pin_15)
- net BORDER_LEDS: now also J15.9 (Pin_9), J14.2 (Pin_2); no longer J16.9 (Pin_9)
- net DIGIT_LEDS: now also J15.8 (Pin_8), J14.1 (Pin_1); no longer J16.8 (Pin_8)
- net GND: now also C1.2, C2.2, C3.2, C4.2, C5.2, C6.2, C7.2, J13.2 (Pin_2), J8.2, J8.SH1 (SHIELD), J8.SH2 (SHIELD), J8.SH3 (SHIELD), J8.SH4 (SHIELD); no longer J12.3 (Pin_3)
- net RELAY_EN: no longer J16.13 (Pin_13)
- net nBLUE_RDY_BTN: now also J15.11 (Pin_11), C7.1, R9.2; no longer J16.11 (Pin_11)
- net nBUZZER_BTN: now also J15.12 (Pin_12), C5.1, R7.2; no longer J16.12 (Pin_12)
- net nPAUSE_BTN: now also J16.11 (Pin_11), C2.1, R4.2; no longer J15.11 (Pin_11)
- net nRED_RDY_BTN: now also J15.10 (Pin_10), C6.1, R8.2; no longer J16.10 (Pin_10)
- net nRESET_BTN: now also J16.12 (Pin_12), C3.1, R5.2; no longer J15.12 (Pin_12)
- net nSTART_BTN: now also J16.10 (Pin_10), C1.1, R3.2; no longer J15.10 (Pin_10)
- net nTIME_SEL: now also J16.13 (Pin_13), C4.1, R6.2; no longer J15.13 (Pin_13)
- net at K1.4: now also J12.3 (Pin_3)
Other:
- note added: "Double Sided Connector"
- note added: "Mounting Screws"
- note added: "Order from LCSC"
- note added: "Order from digikey"
- note added: "Relay Output"
- note removed: "Power Input"
- moved on the sheet: D40, J12, K1A, Q1, R2
