File: ReadyButtonBoard/ReadyButtonBoard.kicad_sch (KiCad schematic)
At the start: 7 parts, among them J2 Conn_01x02_Socket

Commit message: finish ready button board and prod files
Parts:
- removed J1: ~, Connector_PinHeader_2.54mm:PinHeader_1x02_P2.54mm_Vertical, symbol Connector:Conn_01x02_Pin
- removed J2: Conn_01x02_Socket, Connector_JST:JST_EH_S2B-EH_1x02_P2.50mm_Horizontal, symbol Connector:Conn_01x02_Socket
- added D1: Red, LED_SMD:LED_0603_1608Metric, symbol Device:LED
- added J1, J2: Conn_01x08_Socket, Connector_PinSocket_2.54mm:PinSocket_1x08_P2.54mm_Vertical, symbol Connector:Conn_01x08_Socket
- added J3: START, Connector_PinHeader_2.54mm:PinHeader_1x02_P2.54mm_Vertical, symbol Connector:Conn_01x02_Pin
- added J9: WAGO, WAGO_2060-452_998-404:2060-452_998-404, symbol Connector:Conn_01x02_Socket
- added R1: 470, Resistor_SMD:R_0603_1608Metric, symbol Device:R_US
- SW1: value ~ -> START; LCSC C5377619 -> C2888699
Connections:
- net GND: now also D1.1 (K), J2.7 (Pin_7), J3.2 (Pin_2), J9.1 (Pin_1)
- net at SW1.2: now also J1.1 (Pin_1), J3.1 (Pin_1)
- new net: D1.2 (A), R1.1
- new net: J1.3 (Pin_3), R1.2
- new net +3.3V: J1.8 (Pin_8)
- new net +5V: J2.8 (Pin_8), J9.2 (Pin_2)
- no-connect marks 0 -> 6
Other:
- note added: "ANTENNA"
- note added: "ESP8266 Module"
- note added: "RST A0 D0 D5 D6 D7 D8 3.3V"
- note added: "TX RX D1 D2 D3 D4 G 5V"
- note added: "WAGO Battery Input"
