File: DisplayBoard/ArenaTimer.kicad_pcb (KiCad board)
At the start: 2 copper layers, 262.2 x 230 mm, 224 parts, among them J1 Blue ready-up, J10 Red ready-up, J11 SPARE_IO, J12 Screw_Terminal_01x03, J13 WAGO, J14 WAGO, J15 Conn_01x15_Socket, J16 Conn_01x15_Socket, J17 SPARE IO, J18 SPARE 3.3V, J19 SPARE 5V, J2 Conn_01x02_Socket, J20 SPARE GND, J21 SPARE GND, J3 Conn_01x02_Pin, J4 GND, J5 5V, J6 GND, J7 5V, J8 PJ-082BH, J9 Conn_01x06_Pin, K1 G5V-2_Split, Q1 BSS138, Q2 BSS138

Commit message: update LCSC PN for fets to match sc-70 footprint on board
Parts:
- D40: value 1N1007, SMA -> 1N4007, SMA
Changed lines of the file:
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@@
 			)
 		)
-		(property "LCSC" "C5224267"
+		(property "LCSC" "C5224279"
 			(at 0 0 0)
 			(unlocked yes)
@@
 			)
 		)
-		(property "Value" "1N1007, SMA"
+		(property "Value" "1N4007, SMA"
 			(at 0 -2.6 0)
 			(layer "B.Fab")
@@
 			)
 		)
-		(property "LCSC" "C5224267"
+		(property "LCSC" "C5224279"
 			(at 0 0 270)
 			(unlocked yes)
