File: PCB Files/ESP32_Lora/ESP32_Lora/ESP32_Lora.kicad_sch (KiCad schematic)
At the start: 46 parts, among them J114 USB_C_Receptacle_USB2.0_14P, J15 Conn_01x15_Socket, J16 Conn_01x15_Socket, J2 Conn_Coaxial_Small, Q1 SS8050, Q2 SS8050, SW1 SW_Push, SW2 SW_Push, U1 Ai-Thinker RA-08H, U3 CP2102N-Axx-xQFN28, U4 ESP32-WROOM-32UE, U5 AP2112K-3.3, U902 CM1213A−02Sx

Commit message: change RADIO_RST pin to avoid conflict, change 100nF EN cap to 10uF to slow rise time for more stability
Parts:
- C11: value 100nF -> 10uF, 25V; footprint Capacitor_SMD:C_0402_1005Metric -> Capacitor_SMD:C_0603_1608Metric; LCSC C1525 -> C96446
Connections:
- net D34 is gone; now on net RADIO_RST: J16.4 (Pin_4), U4.6 (IO34)
- net RADIO_RST: no longer J16.12 (Pin_12), U4.14 (IO12)
- new net D12: J16.12 (Pin_12), U4.14 (IO12)
Changed lines of the file:
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@@
 		)
 	)
-	(label "RADIO_RST"
+	(label "D12"
 		(at 53.34 227.33 0)
 		(effects
@@
 		)
 	)
-	(label "D34"
+	(label "RADIO_RST"
 		(at 53.34 207.01 0)
 		(effects
@@
 		)
 	)
-	(label "D34"
+	(label "RADIO_RST"
 		(at 386.08 205.74 180)
 		(effects
@@
 		)
 	)
-	(label "RADIO_RST"
+	(label "D12"
 		(at 386.08 165.1 180)
 		(effects
@@
 	)
 	(symbol
+		(lib_id "Device:C")
+		(at 215.9 204.47 0)
+		(unit 1)
+		(body_style 1)
+		(exclude_from_sim no)
+		(in_bom yes)
+		(on_board yes)
+		(in_pos_files yes)
+		(dnp no)
+		(fields_autoplaced yes)
+		(property "Reference" "C11"
+			(at 219.71 203.1999 0)
+			(show_name no)
+			(do_not_autoplace no)
+			(effects
+				(font
+					(size 1.27 1.27)
+				)
+				(justify left)
+			)
+		)
+		(property "Value" "10uF, 25V"
+			(at 219.71 205.7399 0)
+			(show_name no)
+			(do_not_autoplace no)
+			(effects
+				(font
+					(size 1.27 1.27)
+				)
+				(justify left)
+			)
+		)
+		(property "Footprint" "Capacitor_SMD:C_0603_1608Metric"
+			(at 216.8652 208.28 0)
+			(hide yes)
+			(show_name no)
+			(do_not_autoplace no)
+			(effects
+				(font
+					(size 1.27 1.27)
+				)
+			)
+		)
+		(property "Datasheet" ""
+			(at 215.9 204.47 0)
+			(hide yes)
+			(show_name no)
+			(do_not_autoplace no)
+			(effects
+				(font
+					(size 1.27 1.27)
+				)
+			)
+		)
+		(property "Description" "Unpolarized capacitor"
+			(at 215.9 204.47 0)
+			(hide yes)
+			(show_name no)
+			(do_not_autoplace no)
+			(effects
+				(font
+					(size 1.27 1.27)
+				)
+			)
+		)
+		(property "LCSC" "C96446"
+			(at 215.9 204.47 0)
+			(hide yes)
+			(show_name no)
+			(do_not_autoplace no)
+			(effects
+				(font
+					(size 1.27 1.27)
+				)
+			)
+		)
+		(property "Manufacturer" ""
+			(at 215.9 204.47 0)
+			(hide yes)
+			(show_name no)
+			(do_not_autoplace no)
+			(effects
+				(font
+					(size 1.27 1.27)
+				)
+			)
+		)
+		(pin "1"
+		)
+		(pin "2"
+		)
+		(instances
+			(project "ESP32_Lora"
+				(path "/3ea10677-c582-47a8-bbd3-817c5fa3f1e5"
+					(reference "C11")
+					(unit 1)
+				)
+			)
+		)
+	)
+	(symbol
 		(lib_id "Device:LED")
 		(at 394.97 170.18 90)
@@
 					(unit 1)
 				)
-			)
-		)
-	)
-	(symbol
-		(lib_id "Device:C")
-		(at 215.9 204.47 0)
-		(unit 1)
-		(body_style 1)
-		(exclude_from_sim no)
-		(in_bom yes)
-		(on_board yes)
-		(in_pos_files yes)
-		(dnp no)
-		(fields_autoplaced yes)
-		(property "Reference" "C11"
-			(at 219.71 203.1999 0)
-			(show_name no)
-			(do_not_autoplace no)
-			(effects
-				(font
-					(size 1.27 1.27)
-				)
-				(justify left)
-			)
-		)
-		(property "Value" "100nF"
-			(at 219.71 205.7399 0)
-			(show_name no)
-			(do_not_autoplace no)
-			(effects
-				(font
-					(size 1.27 1.27)
-				)
-				(justify left)
-			)
-		)
-		(property "Footprint" "Capacitor_SMD:C_0402_1005Metric"
-			(at 216.8652 208.28 0)
-			(hide yes)
-			(show_name no)
-			(do_not_autoplace no)
-			(effects
-				(font
-					(size 1.27 1.27)
-				)
-			)
-		)
-		(property "Datasheet" ""
-			(at 215.9 204.47 0)
-			(hide yes)
-			(show_name no)
-			(do_not_autoplace no)
-			(effects
-				(font
-					(size 1.27 1.27)
-				)
-			)
-		)
-		(property "Description" "Unpolarized capacitor"
-			(at 215.9 204.47 0)
-			(hide yes)
-			(show_name no)
-			(do_not_autoplace no)
-			(effects
-				(font
-					(size 1.27 1.27)
-				)
-			)
-		)
-		(property "LCSC" "C1525"
-			(at 215.9 204.47 0)
-			(hide yes)
-			(show_name no)
-			(do_not_autoplace no)
-			(effects
-				(font
-					(size 1.27 1.27)
-				)
-			)
-		)
-		(property "Manufacturer" ""
-			(at 215.9 204.47 0)
-			(hide yes)
-			(show_name no)
-			(do_not_autoplace no)
-			(effects
-				(font
-					(size 1.27 1.27)
-				)
-			)
-		)
-		(pin "1"
-		)
-		(pin "2"
-		)
-		(instances
-			(project "ESP32_Lora"
-				(path "/3ea10677-c582-47a8-bbd3-817c5fa3f1e5"
-					(reference "C11")
-					(unit 1)
-				)
