File: PCB Files/TimerRemote/TimerRemote.kicad_sch (KiCad schematic)
At the start: 34 parts, among them J13 WAGO, J2 PROG, J3 VBAT, J5 GND, SW1 START, SW2 PAUSE, SW3 RESET, SW4 TIME_SEL, SW5 BUZZER, SW6 BUZZER, SW7 SW_SPDT, SW8 SW_Push, U1 Ai-Thinker RA-08H, U2 STM32G030K6Tx, U5 AP2112K-3.3

Commit message: get radios working and some other schematic changes in for next rev
Parts:
- removed JP1: Jumper_2_Bridged, Jumper:SolderJumper-2_P1.3mm_Bridged_RoundedPad1.0x1.5mm, symbol Jumper:Jumper_2_Bridged
- added J4: RAD_PROG, Connector_Harwin:Harwin_M20-89006xx_1x06_P2.54mm_Horizontal, symbol Connector:Conn_01x06_Pin
- added R20: 10k, 1%, Resistor_SMD:R_0402_1005Metric, symbol Device:R_US
- J2: value PROG -> STM_PROG
Connections:
- net GND: now also J4.6 (Pin_6), R20.2
- net MCU_UART_RX: now also J4.5 (Pin_5)
- net VBAT: now also J4.1 (Pin_1)
- net RADIO_UART_TX: now reaches U1.12 (RXD/IO16)
- net RADIO_UART_TX: now also J4.4 (Pin_4)
- net RADIO_BOOT: now reaches U1.15 (IO2/BOOT)
- net RADIO_BOOT: now also J4.3 (Pin_3), R20.1
Other:
- note added: "Radio Programmer"
- note added: "STM32 Programmer"
- note removed: "Programmer"
